File: Platinen/MosfetTreiber/JugendNetzteil.brd (EAGLE design)
At the start: 99.5 x 79.5 mm, 69 parts, among them P2 5566-10, Q1 IRF9530, Q2 IRF9530, U1 BSS123, U2 BSS123, U3 BSS123, U4 BSS123, U5 BSS123, U6 BSS123

Commit message: update
Parts:
- C29: value 10nF -> 101F
- C5: value 10nF -> 1nF
- D1, D2, D3, D5, D6, D8: value (none) -> 1n4148
- L1: value (none) -> 1m
- L3: value (none) -> 6m8
- R11: value 10kR -> 2k
- R12: value 10kR -> 10k
- R13: value (none) -> 200
- R3: value (none) -> 2k
- R4: value (none) -> 10k
- R8: value (none) -> 3k9
- R9: value 3k9R -> 3k9
