File: Platinen/MosfetTreiberV2.0/JugendNetzteil.brd (EAGLE design)
At the start: 99.5 x 79.5 mm, 63 parts, among them Q1 IRF9530, Q2 BSS123, Q3 IRLL014N, Q4 BSS123, Q5 IRF9530, Q6 BSS123, Q7 IRLL014N, Q8 BSS123, X1 5566-10

Commit message: Mosfet Treiber fertig gestellt
Parts:
- added U$3: (no value), logo:EAGLE-PLC-8MM
- added U$4: (no value), logo:ESD_10.00
- added U$5: (no value), logo:MUELLTONNE_10.00
- moved C16 2.84 mm to (8.26, 27.3)
- moved C17 2.62 mm to (10.2, 27.3)
Routing:
- net SENS_1A: track 116.7 -> 146.8 mm
- net SENS_2A: track 113.1 -> 143.2 mm
- net SENS_2B: track 36.4 -> 49.3 mm
- net V+: track 602.8 -> 610.2 mm
- net N$18: track 64.5 -> 67.2 mm
- net N$6: track 207.1 -> 205.6 mm
- net N$16: track 198.4 -> 197.7 mm
Other:
- board text added: "PWM"
- board text removed: "PWM IN"
